Commit message: zimmer description package

File: zimmer_test_description/urdf/zimmer_test.xacro (robot description, xacro)
@@ -1,7 +1,7 @@
 <?xml version="1.0" ?>
-<robot name="ZIMMER_test" xmlns:xacro="http://www.ros.org/wiki/xacro">
-<xacro:include filename="$(find ZIMMER_test_description)/urdf/materials.xacro" />
-<xacro:include filename="$(find ZIMMER_test_description)/urdf/ZIMMER_test.trans" />
-<xacro:include filename="$(find ZIMMER_test_description)/urdf/ZIMMER_test.gazebo" />
+<robot name="zimmer_test" xmlns:xacro="http://www.ros.org/wiki/xacro">
+<xacro:include filename="$(find zimmer_test_description)/urdf/materials.xacro" />
+<xacro:include filename="$(find zimmer_test_description)/urdf/zimmer_test.trans" />
+<xacro:include filename="$(find zimmer_test_description)/urdf/zimmer_test.gazebo" />
 <link name="base_link">
   <inertial>
@@ -13,5 +13,5 @@
     <origin xyz="0 0 0" rpy="0 0 0"/>
     <geometry>
-      <mesh filename="file://$(find ZIMMER_test_description)/meshes/base_link.stl" scale="0.001 0.001 0.001"/>
+      <mesh filename="file://$(find zimmer_test_description)/meshes/base_link.stl" scale="0.001 0.001 0.001"/>
     </geometry>
     <material name="silver"/>
@@ -20,5 +20,5 @@
     <origin xyz="0 0 0" rpy="0 0 0"/>
     <geometry>
-      <mesh filename="file://$(find ZIMMER_test_description)/meshes/base_link.stl" scale="0.001 0.001 0.001"/>
+      <mesh filename="file://$(find zimmer_test_description)/meshes/base_link.stl" scale="0.001 0.001 0.001"/>
     </geometry>
   </collision>
@@ -33,5 +33,5 @@
     <origin xyz="-0.0 0.01225 -0.0905" rpy="0 0 0"/>
     <geometry>
-      <mesh filename="file://$(find ZIMMER_test_description)/meshes/SLIDER_1.stl" scale="0.001 0.001 0.001"/>
+      <mesh filename="file://$(find zimmer_test_description)/meshes/SLIDER_1.stl" scale="0.001 0.001 0.001"/>
     </geometry>
     <material name="silver"/>
@@ -40,5 +40,5 @@
     <origin xyz="-0.0 0.01225 -0.0905" rpy="0 0 0"/>
     <geometry>
-      <mesh filename="file://$(find ZIMMER_test_description)/meshes/SLIDER_1.stl" scale="0.001 0.001 0.001"/>
+      <mesh filename="file://$(find zimmer_test_description)/meshes/SLIDER_1.stl" scale="0.001 0.001 0.001"/>
     </geometry>
   </collision>
@@ -53,5 +53,5 @@
     <origin xyz="-0.0 -0.01225 -0.0905" rpy="0 0 0"/>
     <geometry>
-      <mesh filename="file://$(find ZIMMER_test_description)/meshes/SLIDER_2.stl" scale="0.001 0.001 0.001"/>
+      <mesh filename="file://$(find zimmer_test_description)/meshes/SLIDER_2.stl" scale="0.001 0.001 0.001"/>
     </geometry>
     <material name="silver"/>
@@ -60,5 +60,5 @@
     <origin xyz="-0.0 -0.01225 -0.0905" rpy="0 0 0"/>
     <geometry>
-      <mesh filename="file://$(find ZIMMER_test_description)/meshes/SLIDER_2.stl" scale="0.001 0.001 0.001"/>
+      <mesh filename="file://$(find zimmer_test_description)/meshes/SLIDER_2.stl" scale="0.001 0.001 0.001"/>
     </geometry>
   </collision>
