Commit message: functional with 'base_link' no prefix

File: zimmer_description/urdf/zimmer_description.xacro (robot description, xacro)
@@ -2,36 +2,43 @@
 <robot name="zimmer_description" xmlns:xacro="http://www.ros.org/wiki/xacro">
 <xacro:include filename="$(find zimmer_description)/urdf/materials.xacro" />
-<!-- <xacro:include filename="$(find zimmer_description)/urdf/zimmer_description.trans" /> -->
-<!-- <xacro:include filename="$(find zimmer_description)/urdf/zimmer_description.gazebo" /> -->
+<xacro:include filename="$(find zimmer_description)/urdf/zimmer_description.trans" />
+<xacro:include filename="$(find zimmer_description)/urdf/zimmer_description.gazebo" />
+<!-- <xacro:property name="gripper_only" value="false"/> -->
+<xacro:arg name="prefix" default=""/>
 <xacro:property name="y_origin" value="0.01225" />
-<link name="base_link">
-  <inertial>
-    <origin xyz="0.0001004407776845725 -3.782256688140103e-16 0.05878685212370678" rpy="0 0 0"/>
-    <mass value="2.9848284063454846"/>
-    <inertia ixx="0.003517" iyy="0.005044" izz="0.002589" ixy="-0.0" iyz="-0.0" ixz="1.1e-05"/>
-  </inertial>
-  <visual>
-    <origin xyz="0 0 0" rpy="0 0 0"/>
-    <geometry>
-      <mesh filename="file://$(find zimmer_description)/meshes/base_link.stl" scale="0.001 0.001 0.001"/>
-    </geometry>
-    <material name="silver"/>
-  </visual>
-  <collision>
-    <origin xyz="0 0 0" rpy="0 0 0"/>
-    <geometry>
-      <mesh filename="file://$(find zimmer_description)/meshes/base_link.stl" scale="0.001 0.001 0.001"/>
-    </geometry>
-  </collision>
-</link>
+<xacro:arg name="parent" default=""/>
+<!-- <link name="base_link"/> -->
+<!-- ZIMMER BASE MACRO -->
+<xacro:macro name="zimmer_base" params="prefix">
+  <link name="$(arg prefix)base_link">
+    <inertial>
+      <origin xyz="0 0 0" rpy="0 0 0"/>
+      <mass value="2.9848284063454846"/>
+      <inertia ixx="0.003517" iyy="0.005044" izz="0.002589" ixy="-0.0" iyz="-0.0" ixz="1.1e-05"/>
+    </inertial>
+    <visual>
+      <origin xyz="0 0 0" rpy="0 0 0"/>
+      <geometry>
+        <mesh filename="file://$(find zimmer_description)/meshes/base_link.stl" scale="0.001 0.001 0.001"/>
+      </geometry>
+      <material name="silver"/>
+    </visual>
+    <collision>
+      <origin xyz="0 0 0" rpy="0 0 0"/>
+      <geometry>
+        <mesh filename="file://$(find zimmer_description)/meshes/base_link.stl" scale="0.001 0.001 0.001"/>
+      </geometry>
+    </collision>
+  </link>
+</xacro:macro>
 <!-- SLIDER MACRO -->
-<xacro:macro name="slider" params="prefix reflect">
-  <link name="slider_${prefix}">
+<xacro:macro name="slider" params="jaw reflect prefix">
+  <link name="slider_${jaw}">
    <inertial>
-    <origin xyz="0 0 0.022639226003290505" rpy="0 0 0"/>
-    <mass value="0.04981450503853536"/>
-    <inertia ixx="1e-06" iyy="2.3e-05" izz="2.4e-05" ixy="-0.0" iyz="-0.0" ixz="0.0"/>
-  </inertial>
-  <visual>
+      <origin xyz="0 0 0.022639226003290505" rpy="0 0 0"/>
+      <mass value="0.04981450503853536"/>
+      <inertia ixx="1e-06" iyy="2.3e-05" izz="2.4e-05" ixy="-0.0" iyz="-0.0" ixz="0.0"/>
+    </inertial>
+    <visual>
       <origin xyz="-0.0 ${y_origin} -0.0905" rpy="0 0 0"/>
       <geometry>
@@ -47,13 +54,19 @@
     </collision>
   </link>
-  <joint name="base_to_slider_${prefix}" type="prismatic">
+  <joint name="slider_${jaw}_joint" type="prismatic">
     <origin xyz="0.0 ${reflect*(y_origin)} 0.0905" rpy="0 0 0"/>
-    <parent link="base_link"/>
-    <child link="slider_${prefix}"/>
+    <parent link="$(arg prefix)base_link"/>
+    <child link="slider_${jaw}"/>
     <axis xyz="1.0 0.0 0.0"/>
     <limit upper="0.0105" lower="-0.0105" effort="100" velocity="100"/>
   </joint>
 </xacro:macro>
-<xacro:slider prefix="1" reflect="1" />
-<xacro:slider prefix="2" reflect="-1" />
+<xacro:macro name="zimmer_gripper" params="
+  prefix
+  parent">
+  <xacro:zimmer_base prefix="$(arg prefix)"/>
+  <xacro:slider jaw="1" reflect="1" prefix="$(arg prefix)" />
+  <xacro:slider jaw="2" reflect="-1" prefix="$(arg prefix)" />
+</xacro:macro>
+<xacro:zimmer_gripper prefix="" parent="$(arg parent)"/>
 </robot>

Commit message: added zimmer_gripper_macro file, working gripper attachment

File: zimmer_description/urdf/zimmer_description.xacro (robot description, xacro)
@@ -3,13 +3,9 @@
 <xacro:include filename="$(find zimmer_description)/urdf/materials.xacro" />
 <xacro:include filename="$(find zimmer_description)/urdf/zimmer_description.trans" />
-<xacro:include filename="$(find zimmer_description)/urdf/zimmer_description.gazebo" />
-<!-- <xacro:property name="gripper_only" value="false"/> -->
-<xacro:arg name="prefix" default=""/>
+<!-- <xacro:include filename="$(find zimmer_description)/urdf/zimmer_description.gazebo" /> -->
 <xacro:property name="y_origin" value="0.01225" />
-<xacro:arg name="parent" default=""/>
-<!-- <link name="base_link"/> -->
 <!-- ZIMMER BASE MACRO -->
-<xacro:macro name="zimmer_base" params="prefix">
-  <link name="$(arg prefix)base_link">
+<xacro:macro name="zimmer_base" params="prefix parent">
+  <link name="${prefix}base_link">
     <inertial>
       <origin xyz="0 0 0" rpy="0 0 0"/>
@@ -31,8 +27,13 @@
     </collision>
   </link>
+  <joint name="${prefix}base_link_joint" type="fixed">
+    <origin xyz="0 0 0" rpy="0 0 0"/>
+    <parent link="${parent}"/>
+    <child link="${prefix}base_link"/>
+  </joint>
 </xacro:macro>
 <!-- SLIDER MACRO -->
 <xacro:macro name="slider" params="jaw reflect prefix">
-  <link name="slider_${jaw}">
+  <link name="${prefix}slider_${jaw}">
    <inertial>
       <origin xyz="0 0 0.022639226003290505" rpy="0 0 0"/>
@@ -48,5 +49,5 @@
     </visual>
     <collision>
-      <origin xyz="-0.0 ${(y_origin)} -0.0905" rpy="0 0 0"/>
+      <origin xyz="-0.0 ${y_origin} -0.0905" rpy="0 0 0"/>
       <geometry>
         <mesh filename="file://$(find zimmer_description)/meshes/SLIDER.stl" scale="0.001 0.001 0.001"/>
@@ -54,19 +55,11 @@
     </collision>
   </link>
-  <joint name="slider_${jaw}_joint" type="prismatic">
+  <joint name="${prefix}slider_${jaw}_joint" type="prismatic">
     <origin xyz="0.0 ${reflect*(y_origin)} 0.0905" rpy="0 0 0"/>
-    <parent link="$(arg prefix)base_link"/>
-    <child link="slider_${jaw}"/>
+    <parent link="${prefix}base_link"/>
+    <child link="${prefix}slider_${jaw}"/>
     <axis xyz="1.0 0.0 0.0"/>
     <limit upper="0.0105" lower="-0.0105" effort="100" velocity="100"/>
   </joint>
 </xacro:macro>
-<xacro:macro name="zimmer_gripper" params="
-  prefix
-  parent">
-  <xacro:zimmer_base prefix="$(arg prefix)"/>
-  <xacro:slider jaw="1" reflect="1" prefix="$(arg prefix)" />
-  <xacro:slider jaw="2" reflect="-1" prefix="$(arg prefix)" />
-</xacro:macro>
-<xacro:zimmer_gripper prefix="" parent="$(arg parent)"/>
 </robot>
