Commit message: workspace URDF with basic camera mount

File: workspace_test/urdf/testing_macro.xacro (robot description, xacro)
@@ -2,4 +2,5 @@
 <robot xmlns:xacro="http://ros.org/wiki/xacro">
   <xacro:include filename="$(find ur_description)/urdf/ur_macro.xacro"/>
+  <xacro:include filename="$(find realsense2_description)/urdf/_d435.urdf.xacro"/>
   <xacro:macro name="my_robot_cell" params="
     parent
@@ -31,4 +32,67 @@
       </collision>
     </link>
+    <!-- CAMERA MOUNT -->
+    <joint name="table_to_camera_mount" type="fixed">
+      <parent link="table"/>
+      <child link="camera_mount"/>
+      <origin xyz="0.24 0.762 0" rpy="0 0 0"/>
+    </joint>
+    <link name="camera_mount">
+      <visual>
+        <geometry>
+          <box size="0.030 0.030 0.9144"/>
+        </geometry>
+        <origin rpy="0 0 0" xyz="0 0 ${0.9144 / 2}"/>
+      </visual>
+      <collision>
+        <geometry>
+          <box size="0.030 0.030 0.9144"/>
+        </geometry>
+        <origin rpy="0 0 0" xyz="0 0 ${0.9144 / 2}"/>
+      </collision>
+    </link>
+    <!-- SECOND LINK -->
+    <link name="camera_mount_2">
+      <visual>
+        <geometry>
+          <box size="0.030 0.030 0.5"/>
+        </geometry>
+        <origin rpy="0 0 0" xyz="0 0 0.25"/>
+      </visual>
+      <collision>
+        <geometry>
+          <box size="0.030 0.030 0.5"/>
+        </geometry>
+        <origin rpy="0 0 0" xyz="0 0 0.25"/>
+      </collision>
+    </link>
+    <joint name="camera_mount_joint" type="fixed">
+      <parent link="camera_mount"/>
+      <child link="camera_mount_2"/>
+      <origin xyz="0 0 0.9144" rpy="${pi/2} 0 0"/>
+    </joint>
+    <!-- CAMERA -->
+    <!-- <xacro:realsense2_camera>
+      <origin xyz="0 0 0.25" rpy="0 0 0"/>
+    </xacro:realsense_d435>
+    <joint name="camera_mount_to_realsense_d435" type="fixed">
+      <parent link="camera_mount_2"/>
+      <child link="realsense_d435"/>
+      <origin xyz="0 0 0.25" rpy="0 0 0"/>
+    </joint> -->
+    <!-- <link name="realsense_d435">
+      <visual>
+        <geometry>
+          <mesh filename="package://realsense2_description/meshes/_d435.dae"/>
+        </geometry>
+        <origin rpy="0 0 0" xyz="0 0 0"/>
+      </visual>
+      <collision>
+        <geometry>
+          <mesh filename="package://realsense2_description/meshes/_d435.dae"/>
+        </geometry>
+        <origin rpy="0 0 0" xyz="0 0 0"/>
+      </collision>
+    </link> -->
     <material name="white">
       <color rgba="1 1 1 1"/>

File: workspace_test/urdf/workspace_urdf.xacro (robot description, xacro)
@@ -2,4 +2,5 @@
 <robot name="my_robot_cell" xmlns:xacro="http://ros.org/wiki/xacro">
   <xacro:include filename="$(find my_robot_cell_description)/urdf/testing_macro.xacro"/>
+  <xacro:include filename="$(find realsense2_description)/urdf/_d435.urdf.xacro"/>
   <xacro:arg name="ur_type" default="ur3e"/>
   <xacro:arg name="joint_limits_parameters_file" default="$(find ur_description)/config/$(arg ur_type)/joint_limits.yaml"/>
@@ -7,4 +8,7 @@
   <xacro:arg name="physical_parameters_file" default="$(find ur_description)/config/$(arg ur_type)/physical_parameters.yaml"/>
   <xacro:arg name="visual_parameters_file" default="$(find ur_description)/config/$(arg ur_type)/visual_parameters.yaml"/>
+  <xacro:arg name="use_nominal_extrinsics" default="true"/>
+  <xacro:arg name="add_plug" default="false"/>
+  <xacro:arg name="use_mesh" default="true"/>
   <link name="world"/>
   <!--This will create the scene where the robot is located in-->
@@ -19,3 +23,25 @@
       <origin xyz="0 0 0.845" rpy="0 0 0" />
   </xacro:my_robot_cell>
+  <!-- <link name="base_link"/>
+    <visual>
+      <geometry>
+        <mesh filename="package://realsense2_description/meshes/d435_base.dae"/>
+      </geometry>
+      <origin xyz="0 0 0" rpy="0 0 0"/>
+    </visual>
+    <collision>
+      <geometry>
+        <mesh filename="package://realsense2_description/meshes/d435_base.dae"/>
+      </geometry>
+      <origin xyz="0 0 0" rpy="0 0 0"/>
+    </collision>
+  </link>
+  <joint name="camera_mount_to_realsense_d435" type="fixed">
+    <parent link="camera_mount_2"/>
+    <child link="base_link"/>
+    <origin xyz="0 0 0.25" rpy="0 0 0"/>
+  </joint>
+  <xacro:sensor_d435 parent="base_link" use_nominal_extrinsics="$(arg use_nominal_extrinsics)" add_plug="$(arg add_plug)" use_mesh="$(arg use_mesh)">
+    <origin xyz="0 0 0" rpy="0 0 0"/>
+  </xacro:sensor_d435> -->
 </robot>

Commit message: Added camera mesh to testing_macro

File: workspace_test/urdf/testing_macro.xacro (robot description, xacro)
@@ -73,16 +73,8 @@
     </joint>
     <!-- CAMERA -->
-    <!-- <xacro:realsense2_camera>
-      <origin xyz="0 0 0.25" rpy="0 0 0"/>
-    </xacro:realsense_d435>
-    <joint name="camera_mount_to_realsense_d435" type="fixed">
-      <parent link="camera_mount_2"/>
-      <child link="realsense_d435"/>
-      <origin xyz="0 0 0.25" rpy="0 0 0"/>
-    </joint> -->
-    <!-- <link name="realsense_d435">
+    <link name="realsense_d435">
       <visual>
         <geometry>
-          <mesh filename="package://realsense2_description/meshes/_d435.dae"/>
+          <mesh filename="package://realsense2_description/meshes/d435.dae"/>
         </geometry>
         <origin rpy="0 0 0" xyz="0 0 0"/>
@@ -90,9 +82,14 @@
       <collision>
         <geometry>
-          <mesh filename="package://realsense2_description/meshes/_d435.dae"/>
+          <mesh filename="package://realsense2_description/meshes/d435.dae"/>
         </geometry>
         <origin rpy="0 0 0" xyz="0 0 0"/>
       </collision>
-    </link> -->
+    </link>
+    <joint name="camera_mount_to_realsense_d435" type="fixed">
+      <parent link="camera_mount_2"/>
+      <child link="realsense_d435"/>
+      <origin xyz="0 -0.04 0.25" rpy="${pi/2} ${3*pi/2} 0"/>
+    </joint>
     <material name="white">
       <color rgba="1 1 1 1"/>

Commit message: workspace_marco defined, testing_macro deleted

File: workspace_test/urdf/testing_macro.xacro (robot description, xacro)
@@ -70,5 +70,6 @@
       <parent link="camera_mount"/>
       <child link="camera_mount_2"/>
-      <origin xyz="0 0 0.9144" rpy="${pi/2} 0 0"/>
+      <!-- edit origin of joints to change camera height -->
+      <origin xyz="0 0 0.8" rpy="${pi/2} 0 0"/>
     </joint>
     <!-- CAMERA -->

File: workspace_test/urdf/workspace_macro.xacro (robot description, xacro)
@@ -2,5 +2,6 @@
 <robot xmlns:xacro="http://ros.org/wiki/xacro">
   <xacro:include filename="$(find ur_description)/urdf/ur_macro.xacro"/>
-  <xacro:macro name="workspace_synbio" params="
+  <xacro:include filename="$(find realsense2_description)/urdf/_d435.urdf.xacro"/>
+  <xacro:macro name="my_robot_cell" params="
     parent
     *origin
@@ -22,5 +23,5 @@
           <mesh filename="package://workspace_test/meshes/workbench.dae"/>
         </geometry>
-        <origin rpy="0 0 0" xyz="0.75 0.5 -1"/>
+        <origin rpy="0 0 0" xyz="0 0.762 -0.845"/>
       </visual>
       <collision>
@@ -28,7 +29,68 @@
           <mesh filename="package://workspace_test/meshes/workbench.dae"/>
         </geometry>
-        <origin rpy="0 0 0" xyz="0.75 0.5 -1"/>
+        <origin rpy="0 0 0" xyz="0 0.762 -0.845"/>
       </collision>
     </link>
+    <!-- CAMERA MOUNT -->
+    <joint name="table_to_camera_mount" type="fixed">
+      <parent link="table"/>
+      <child link="camera_mount"/>
+      <origin xyz="0.24 0.762 0" rpy="0 0 0"/>
+    </joint>
+    <link name="camera_mount">
+      <visual>
+        <geometry>
+          <box size="0.030 0.030 0.9144"/>
+        </geometry>
+        <origin rpy="0 0 0" xyz="0 0 ${0.9144 / 2}"/>
+      </visual>
+      <collision>
+        <geometry>
+          <box size="0.030 0.030 0.9144"/>
+        </geometry>
+        <origin rpy="0 0 0" xyz="0 0 ${0.9144 / 2}"/>
+      </collision>
+    </link>
+    <!-- SECOND LINK -->
+    <link name="camera_mount_2">
+      <visual>
+        <geometry>
+          <box size="0.030 0.030 0.5"/>
+        </geometry>
+        <origin rpy="0 0 0" xyz="0 0 0.25"/>
+      </visual>
+      <collision>
+        <geometry>
+          <box size="0.030 0.030 0.5"/>
+        </geometry>
+        <origin rpy="0 0 0" xyz="0 0 0.25"/>
+      </collision>
+    </link>
+    <joint name="camera_mount_joint" type="fixed">
+      <parent link="camera_mount"/>
+      <child link="camera_mount_2"/>
+      <!-- edit origin of joints to change camera height -->
+      <origin xyz="0 0 0.8" rpy="${pi/2} 0 0"/>
+    </joint>
+    <!-- CAMERA -->
+    <link name="realsense_d435">
+      <visual>
+        <geometry>
+          <mesh filename="package://realsense2_description/meshes/d435.dae"/>
+        </geometry>
+        <origin rpy="0 0 0" xyz="0 0 0"/>
+      </visual>
+      <collision>
+        <geometry>
+          <mesh filename="package://realsense2_description/meshes/d435.dae"/>
+        </geometry>
+        <origin rpy="0 0 0" xyz="0 0 0"/>
+      </collision>
+    </link>
+    <joint name="camera_mount_to_realsense_d435" type="fixed">
+      <parent link="camera_mount_2"/>
+      <child link="realsense_d435"/>
+      <origin xyz="0 -0.04 0.25" rpy="${pi/2} ${3*pi/2} 0"/>
+    </joint>
     <material name="white">
       <color rgba="1 1 1 1"/>
@@ -38,6 +100,7 @@
       <visual>
         <geometry>
-          <mesh filename="package://my_robot_cell_description/meshes/wall.dae"/>
+          <box size="4.44 0.1 2.5"/>
         </geometry>
+        <material name="white"/>
       </visual>
       <collision>
@@ -50,12 +113,12 @@
       <parent link="table"/>
       <child link="wall"/>
-      <origin xyz="1 1.5 0.5"/>
+      <origin xyz="1 1.1 0.5"/>
     </joint>
     <!-- ROBOT MOUNT 1 -->
-    <link name="robot_mount"/>
-    <joint name="base_to_robot_mount" type="fixed">
+    <link name="robot_mount_1"/>
+    <joint name="base_to_robot_mount_1" type="fixed">
       <parent link="table"/>
-      <child link="robot_mount"/>
-      <origin xyz="0.845 0.85 0" rpy="0 0 ${pi}" />
+      <child link="robot_mount_1"/>
+      <origin xyz="0.9144 0.5588 0" rpy="0 0 ${3*pi/2}" />
     </joint>
     <!--This will create the specific robot-->
@@ -63,5 +126,5 @@
       name="${ur_type}"
       tf_prefix="${ur_type}1_"
-      parent="robot_mount"
+      parent="robot_mount_1"
       joint_limits_parameters_file="${joint_limits_parameters_file}"
       kinematics_parameters_file="${kinematics_parameters_file}"
@@ -72,9 +135,9 @@
     </xacro:ur_robot>
     <!-- ROBOT MOUNT 2 -->
-    <link name="robot_mount"/>
-    <joint name="base_to_robot_mount" type="fixed">
+    <link name="robot_mount_2"/>
+    <joint name="base_to_robot_mount_2" type="fixed">
       <parent link="table"/>
-      <child link="robot_mount"/>
-      <origin xyz="1.2 0.5 0" rpy="0 0 ${pi}" />
+      <child link="robot_mount_2"/>
+      <origin xyz="1.5748 0.508 0" rpy="0 0 ${3*pi/2}" />
     </joint>
     <!-- ROBOT 2 -->
@@ -82,5 +145,5 @@
       name="${ur_type}"
       tf_prefix="${ur_type}2_"
-      parent="robot_mount"
+      parent="robot_mount_2"
       joint_limits_parameters_file="${joint_limits_parameters_file}"
       kinematics_parameters_file="${kinematics_parameters_file}"

File: workspace_test/urdf/workspace_urdf.xacro (robot description, xacro)
@@ -23,24 +23,7 @@
       <origin xyz="0 0 0.845" rpy="0 0 0" />
   </xacro:my_robot_cell>
-  <!-- <link name="base_link"/>
-    <visual>
-      <geometry>
-        <mesh filename="package://realsense2_description/meshes/d435_base.dae"/>
-      </geometry>
-      <origin xyz="0 0 0" rpy="0 0 0"/>
-    </visual>
-    <collision>
-      <geometry>
-        <mesh filename="package://realsense2_description/meshes/d435_base.dae"/>
-      </geometry>
-      <origin xyz="0 0 0" rpy="0 0 0"/>
-    </collision>
-  </link>
-  <joint name="camera_mount_to_realsense_d435" type="fixed">
-    <parent link="camera_mount_2"/>
-    <child link="base_link"/>
-    <origin xyz="0 0 0.25" rpy="0 0 0"/>
-  </joint>
-  <xacro:sensor_d435 parent="base_link" use_nominal_extrinsics="$(arg use_nominal_extrinsics)" add_plug="$(arg add_plug)" use_mesh="$(arg use_mesh)">
+  <!-- uncomment to test sensor macro -->
+  <!-- <link name="realsense_d435"/>
+  <xacro:sensor_d435 parent="realsense_d435" use_nominal_extrinsics="$(arg use_nominal_extrinsics)" add_plug="$(arg add_plug)" use_mesh="$(arg use_mesh)">
     <origin xyz="0 0 0" rpy="0 0 0"/>
   </xacro:sensor_d435> -->
