Commit message: Corrected sensor position for URDF

File: workspace_test/urdf/workspace_macro.xacro (robot description, xacro)
@@ -71,13 +71,13 @@
       <child link="camera_mount_2"/>
       <!-- edit origin of joints to change camera height -->
-      <origin xyz="0 0 0.8" rpy="${pi/2} 0 0"/>
+      <origin xyz="0 0 0.690875" rpy="${pi/2} 0 0"/>
     </joint>
     <!-- CAMERA -->
-    <link name="realsense_d435">
+    <link name="camera_link">
       <visual>
         <geometry>
           <mesh filename="package://realsense2_description/meshes/d435.dae"/>
         </geometry>
-        <origin rpy="0 0 0" xyz="0 0 0"/>
+        <origin rpy="0 ${pi/2} 0" xyz="0 0 0"/>
       </visual>
       <collision>
@@ -85,11 +85,11 @@
           <mesh filename="package://realsense2_description/meshes/d435.dae"/>
         </geometry>
-        <origin rpy="0 0 0" xyz="0 0 0"/>
+        <origin rpy="$0 ${pi/2} 0" xyz="0 0 0"/>
       </collision>
     </link>
     <joint name="camera_mount_to_realsense_d435" type="fixed">
       <parent link="camera_mount_2"/>
-      <child link="realsense_d435"/>
-      <origin xyz="0 -0.04 0.25" rpy="${pi/2} ${3*pi/2} 0"/>
+      <child link="camera_link"/>
+      <origin xyz="0 -0.04 0.25" rpy="0 0 ${3*pi/2}"/>
     </joint>
     <material name="white">

File: workspace_test/urdf/workspace_urdf.xacro (robot description, xacro)
@@ -24,7 +24,7 @@
   </xacro:my_robot_cell>
   <!-- uncomment to test sensor macro -->
-  <!-- <link name="realsense_d435"/>
-  <xacro:sensor_d435 parent="realsense_d435" use_nominal_extrinsics="$(arg use_nominal_extrinsics)" add_plug="$(arg add_plug)" use_mesh="$(arg use_mesh)">
+  <!-- <link name="camera_link"/> -->
+  <xacro:sensor_d435 parent="camera_link" use_nominal_extrinsics="$(arg use_nominal_extrinsics)" add_plug="$(arg add_plug)" use_mesh="$(arg use_mesh)">
     <origin xyz="0 0 0" rpy="0 0 0"/>
-  </xacro:sensor_d435> -->
+  </xacro:sensor_d435>
 </robot>

Commit message: Small positional adjustments, added Octomap to pkg.xml

File: workspace_test/urdf/workspace_macro.xacro (robot description, xacro)
@@ -85,5 +85,5 @@
           <mesh filename="package://realsense2_description/meshes/d435.dae"/>
         </geometry>
-        <origin rpy="$0 ${pi/2} 0" xyz="0 0 0"/>
+        <origin rpy="0 ${pi/2} 0" xyz="0 0 0"/>
       </collision>
     </link>
@@ -91,5 +91,5 @@
       <parent link="camera_mount_2"/>
       <child link="camera_link"/>
-      <origin xyz="0 -0.04 0.25" rpy="0 0 ${3*pi/2}"/>
+      <origin xyz="0 -0.04 0.3375" rpy="${pi/2} 0 ${3*pi/2}"/>
     </joint>
     <material name="white">

File: workspace_test/urdf/workspace_urdf.xacro (robot description, xacro)
@@ -1,5 +1,5 @@
 <?xml version="1.0"?>
 <robot name="my_robot_cell" xmlns:xacro="http://ros.org/wiki/xacro">
-  <xacro:include filename="$(find my_robot_cell_description)/urdf/testing_macro.xacro"/>
+  <xacro:include filename="$(find my_robot_cell_description)/urdf/workspace_macro.xacro"/>
   <xacro:include filename="$(find realsense2_description)/urdf/_d435.urdf.xacro"/>
   <xacro:arg name="ur_type" default="ur3e"/>

Commit message: Changed to Realsense Macro

File: workspace_test/urdf/workspace_macro.xacro (robot description, xacro)
@@ -3,4 +3,7 @@
   <xacro:include filename="$(find ur_description)/urdf/ur_macro.xacro"/>
   <xacro:include filename="$(find realsense2_description)/urdf/_d435.urdf.xacro"/>
+  <xacro:arg name="use_nominal_extrinsics" default="true"/>
+  <xacro:arg name="add_plug" default="false"/>
+  <xacro:arg name="use_mesh" default="true"/>
   <xacro:macro name="my_robot_cell" params="
     parent
@@ -33,10 +36,10 @@
     </link>
     <!-- CAMERA MOUNT -->
-    <joint name="table_to_camera_mount" type="fixed">
+    <joint name="table_to_camera_mount_1" type="fixed">
       <parent link="table"/>
-      <child link="camera_mount"/>
+      <child link="camera_mount_1"/>
       <origin xyz="0.24 0.762 0" rpy="0 0 0"/>
     </joint>
-    <link name="camera_mount">
+    <link name="camera_mount_1">
       <visual>
         <geometry>
@@ -68,28 +71,19 @@
     </link>
     <joint name="camera_mount_joint" type="fixed">
-      <parent link="camera_mount"/>
+      <parent link="camera_mount_1"/>
       <child link="camera_mount_2"/>
       <!-- edit origin of joints to change camera height -->
-      <origin xyz="0 0 0.690875" rpy="${pi/2} 0 0"/>
+      <origin xyz="0 0 0.8" rpy="${pi/2} 0 0"/>
     </joint>
+<!-- 0.690875 -->
     <!-- CAMERA -->
-    <link name="camera_link">
-      <visual>
-        <geometry>
-          <mesh filename="package://realsense2_description/meshes/d435.dae"/>
-        </geometry>
-        <origin rpy="0 ${pi/2} 0" xyz="0 0 0"/>
-      </visual>
-      <collision>
-        <geometry>
-          <mesh filename="package://realsense2_description/meshes/d435.dae"/>
-        </geometry>
-        <origin rpy="0 ${pi/2} 0" xyz="0 0 0"/>
-      </collision>
-    </link>
+    <link name="camera_mount_3" />
+    <xacro:sensor_d435 parent="camera_mount_3" use_nominal_extrinsics="$(arg use_nominal_extrinsics)" add_plug="$(arg add_plug)" use_mesh="$(arg use_mesh)">
+      <origin xyz="0 0 0" rpy="0 0 0"/>
+    </xacro:sensor_d435>
     <joint name="camera_mount_to_realsense_d435" type="fixed">
       <parent link="camera_mount_2"/>
-      <child link="camera_link"/>
-      <origin xyz="0 -0.04 0.3375" rpy="${pi/2} 0 ${3*pi/2}"/>
+      <child link="camera_mount_3"/>
+      <origin xyz="0.01 -0.025 0.3375" rpy="${pi/2} 0 ${3*pi/2}"/>
     </joint>
     <material name="white">
