Commit message: Working left arm. Fixed XACRO

File: synbio_control/urdf/synbio_env_controlled.urdf.xacro (robot description, xacro)
@@ -2,6 +2,4 @@
 <robot name="synbio_env" xmlns:xacro="http://ros.org/wiki/xacro">
   <xacro:include filename="$(find workspace_test)/urdf/env_macro.xacro"/>
-  <xacro:include filename="$(find workspace_test)/urdf/left_robot.urdf.xacro"/>
-  <xacro:include filename="$(find workspace_test)/urdf/right_robot.urdf.xacro"/>
   <xacro:include filename="$(find ur_description)/urdf/ur.ros2_control.xacro"/>
   <xacro:include filename="$(find ur_description)/urdf/ur_macro.xacro"/>
@@ -16,5 +14,5 @@
   <xacro:arg name="ur_input_recipe_filename" default="$(find ur_robot_driver)/resources/rtde_input_recipe.txt"/>
   <!-- LEFT -->
-  <xacro:property name="left_xyz" default="1.5748 0.508 0.845" />
+  <xacro:property name="left_xyz" default="0.9144 0.5588 0.845" />
   <xacro:property name="left_rpy" default="0 0 ${3*pi/2}" />
   <xacro:property name="left_tf_prefix" default="left_"/>
@@ -33,5 +31,5 @@
   <!-- RIGHT -->
   <xacro:property name="right_xyz" default="1.5748 0.508 0.845"/>
-  <xacro:property name="right_rpy" default="0 0 ${3*pi/2}" />
+  <xacro:property name="right_rpy" default="0 0 ${pi}" />
   <xacro:property name="right_tf_prefix" default="right_"/>
   <!-- <xacro:arg name="right_ur_type" default="ur3e"/>
@@ -75,24 +73,3 @@
     <origin xyz="${left_xyz}" rpy="${left_rpy}"/>
   </xacro:ur_robot>
-  <!-- <xacro:left_robot_macro
-    parent="world"
-    left_ur_type="$(arg left_ur_type)"
-    left_joint_limits_parameters_file="$(arg left_joint_limits_parameters_file)"
-    left_kinematics_parameters_file="$(arg left_kinematics_parameters_file)"
-    left_physical_parameters_file="$(arg left_physical_parameters_file)"
-    left_visual_parameters_file="$(arg left_visual_parameters_file)"
-    left_generate_ros2_control_tag="$(arg left_generate_ros2_control_tag)"
-    >
-    <origin xyz="0 0 1" rpy="0 0 0" />
-  </xacro:left_robot_macro> -->
-  <!-- <xacro:right_robot_macro
-    parent="world"
-    right_ur_type="$(arg right_ur_type)"
-    right_joint_limits_parameters_file="$(arg right_joint_limits_parameters_file)"
-    right_kinematics_parameters_file="$(arg right_kinematics_parameters_file)"
-    right_physical_parameters_file="$(arg right_physical_parameters_file)"
-    right_visual_parameters_file="$(arg right_visual_parameters_file)"
-    >
-    <origin xyz="0 0 1" rpy="0 0 0" />
-  </xacro:right_robot_macro> -->
 </robot>

Commit message: Working dual arm control

File: synbio_control/urdf/synbio_env_controlled.urdf.xacro (robot description, xacro)
@@ -24,5 +24,4 @@
   <!-- LEFT CONTROL PARAMS -->
   <xacro:arg name="left_robot_ip" default="0.0.0.0"/>
-  <xacro:arg name="left_headless_mode" default="false" />
   <xacro:arg name="left_reverse_port" default="50001"/>
   <xacro:arg name="left_script_sender_port" default="50002"/>
@@ -33,17 +32,15 @@
   <xacro:property name="right_rpy" default="0 0 ${pi}" />
   <xacro:property name="right_tf_prefix" default="right_"/>
-  <!-- <xacro:arg name="right_ur_type" default="ur3e"/>
+  <xacro:arg name="right_ur_type" default="ur3e"/>
   <xacro:arg name="right_joint_limits_parameters_file" default="$(find ur_description)/config/$(arg right_ur_type)/joint_limits.yaml"/>
   <xacro:arg name="right_kinematics_parameters_file" default="$(find ur_description)/config/$(arg right_ur_type)/default_kinematics.yaml"/>
   <xacro:arg name="right_physical_parameters_file" default="$(find ur_description)/config/$(arg right_ur_type)/physical_parameters.yaml"/>
-  <xacro:arg name="right_visual_parameters_file" default="$(find ur_description)/config/$(arg right_ur_type)/visual_parameters.yaml"/> -->
+  <xacro:arg name="right_visual_parameters_file" default="$(find ur_description)/config/$(arg right_ur_type)/visual_parameters.yaml"/>
   <!-- RIGHT CONTROL PARAMS -->
-  <!-- <xacro:arg name="right_robot_ip" default="0.0.0.0"/>
-  <xacro:arg name="right_headless_mode" default="false" />
-  <xacro:arg name="right_ur_script_filename" default="$(find ur_client_library)/resources/external_control.urscript"/>
-  <xacro:arg name="right_ur_output_recipe_filename" default="$(find ur_robot_driver)/resources/rtde_output_recipe.txt"/>
-  <xacro:arg name="right_ur_input_recipe_filename" default="$(find ur_robot_driver)/resources/rtde_input_recipe.txt"/>
-  <xacro:arg name="right_use_mock_hardware" default="false" />
-  <xacro:arg name="right_mock_sensor_commands" default="false" /> -->
+  <xacro:arg name="right_robot_ip" default="0.0.0.0"/>
+  <xacro:arg name="right_reverse_port" default="50005"/>
+  <xacro:arg name="right_script_sender_port" default="50006"/>
+  <xacro:arg name="right_script_command_port" default="50008"/>
+  <xacro:arg name="right_trajectory_port" default="50007"/>
   <xacro:property name="table_height" value="0.845"/>
   <link name="world"/>
@@ -57,5 +54,5 @@
     parent="world"
     tf_prefix="${left_tf_prefix}"
-    name="$(arg left_ur_type)"
+    name="left_$(arg left_ur_type)"
     robot_ip="$(arg left_robot_ip)"
     joint_limits_parameters_file="$(arg left_joint_limits_parameters_file)"
@@ -70,6 +67,33 @@
     use_fake_hardware="$(arg use_fake_hardware)"
     fake_sensor_commands="$(arg fake_sensor_commands)"
+    reverse_port="$(arg left_reverse_port)"
+    script_command_port="$(arg left_script_command_port)"
+    script_sender_port="$(arg left_script_sender_port)"
+    trajectory_port="$(arg left_trajectory_port)"
     >
     <origin xyz="${left_xyz}" rpy="${left_rpy}"/>
   </xacro:ur_robot>
+  <xacro:ur_robot
+    parent="world"
+    tf_prefix="${right_tf_prefix}"
+    name="right_$(arg right_ur_type)"
+    robot_ip="$(arg right_robot_ip)"
+    joint_limits_parameters_file="$(arg right_joint_limits_parameters_file)"
+    kinematics_parameters_file="$(arg right_kinematics_parameters_file)"
+    physical_parameters_file="$(arg right_physical_parameters_file)"
+    visual_parameters_file="$(arg right_visual_parameters_file)"
+    generate_ros2_control_tag="$(arg generate_ros2_control_tag)"
+    script_filename="$(arg ur_script_filename)"
+    input_recipe_filename="$(arg ur_input_recipe_filename)"
+    output_recipe_filename="$(arg ur_output_recipe_filename)"
+    non_blocking_read="$(arg non_blocking_read)"
+    use_fake_hardware="$(arg use_fake_hardware)"
+    fake_sensor_commands="$(arg fake_sensor_commands)"
+    reverse_port="$(arg right_reverse_port)"
+    script_command_port="$(arg right_script_command_port)"
+    script_sender_port="$(arg right_script_sender_port)"
+    trajectory_port="$(arg right_trajectory_port)"
+    >
+    <origin xyz="${right_xyz}" rpy="${right_rpy}"/>
+  </xacro:ur_robot>
 </robot>

Commit message: Fixed spacing

File: synbio_control/urdf/synbio_env_controlled.urdf.xacro (robot description, xacro)
@@ -15,5 +15,5 @@
   <!-- LEFT -->
   <xacro:property name="left_xyz" default="0.9144 0.5588 0.845" />
-  <xacro:property name="left_rpy" default="0 0 ${3*pi/2}" />
+  <xacro:property name="left_rpy" default="0 0 ${pi}" />
   <xacro:property name="left_tf_prefix" default="left_"/>
   <xacro:arg name="left_ur_type" default="ur3e"/>

File: workspace_test/urdf/env_macro.xacro (robot description, xacro)
@@ -1,5 +1,4 @@
 <?xml version="1.0"?>
 <robot xmlns:xacro="http://ros.org/wiki/xacro">
-  <xacro:include filename="$(find ur_description)/urdf/ur_macro.xacro"/>
   <xacro:include filename="$(find realsense2_description)/urdf/_d435.urdf.xacro"/>
   <xacro:arg name="use_nominal_extrinsics" default="true"/>
@@ -102,5 +101,5 @@
       <parent link="table"/>
       <child link="wall"/>
-      <origin xyz="1 1.1 0.5"/>
+      <origin xyz="1 0.85 0.5"/>
     </joint>
   </xacro:macro>

Commit message: Removed workbench from URDF

File: synbio_control/urdf/synbio_env_controlled.urdf.xacro (robot description, xacro)
@@ -4,4 +4,5 @@
   <xacro:include filename="$(find ur_description)/urdf/ur.ros2_control.xacro"/>
   <xacro:include filename="$(find ur_description)/urdf/ur_macro.xacro"/>
+  <xacro:property name="table_height" value="0"/>
   <!-- SHARED CONTROL PARAMS -->
   <xacro:arg name="use_fake_hardware" default="false" />
@@ -14,5 +15,5 @@
   <xacro:arg name="ur_input_recipe_filename" default="$(find ur_robot_driver)/resources/rtde_input_recipe.txt"/>
   <!-- LEFT -->
-  <xacro:property name="left_xyz" default="0.9144 0.5588 0.845" />
+  <xacro:property name="left_xyz" default="0.9144 0.5588 ${table_height}" />
   <xacro:property name="left_rpy" default="0 0 ${pi}" />
   <xacro:property name="left_tf_prefix" default="left_"/>
@@ -29,5 +30,5 @@
   <xacro:arg name="left_trajectory_port" default="50003"/>
   <!-- RIGHT -->
-  <xacro:property name="right_xyz" default="1.5748 0.508 0.845"/>
+  <xacro:property name="right_xyz" default="1.5748 0.508 ${table_height}"/>
   <xacro:property name="right_rpy" default="0 0 ${pi}" />
   <xacro:property name="right_tf_prefix" default="right_"/>
@@ -43,5 +44,4 @@
   <xacro:arg name="right_script_command_port" default="50008"/>
   <xacro:arg name="right_trajectory_port" default="50007"/>
-  <xacro:property name="table_height" value="0.845"/>
   <link name="world"/>
   <!--This will create the scene where the robot is located in-->

File: workspace_test/urdf/env_macro.xacro (robot description, xacro)
@@ -18,20 +18,24 @@
       <visual>
         <geometry>
-          <mesh filename="package://workspace_test/meshes/workbench.dae"/>
+          <box size="1.8288 0.762 0.0445"/>
         </geometry>
-        <origin rpy="0 0 0" xyz="0 0.762 -0.845"/>
+        <material name="gray">
+          <color rgba="0.5 0.5 0.5 1"/>
+        </material>
+        <origin rpy="0 0 0" xyz="${1.8288 / 2} ${0.762 / 2} ${-0.0445 / 2}"/>
       </visual>
       <collision>
         <geometry>
-          <mesh filename="package://workspace_test/meshes/workbench.dae"/>
+          <box size="1.8288 0.762 0.0445"/>
         </geometry>
-        <origin rpy="0 0 0" xyz="0 0.762 -0.845"/>
+        <origin rpy="0 0 0" xyz="${1.8288 / 2} ${0.762 / 2} ${-0.0445 / 2}"/>
       </collision>
     </link>
+    <!-- <mesh filename="package://workspace_test/meshes/workbench.dae"/> -->
     <!-- CAMERA MOUNT -->
     <joint name="table_to_camera_mount_1" type="fixed">
       <parent link="table"/>
       <child link="camera_mount_1"/>
-      <origin xyz="0.24 0.762 0" rpy="0 0 0"/>
+      <origin xyz="0.25 0.762 0" rpy="0 0 0"/>
     </joint>
     <link name="camera_mount_1">
@@ -40,5 +44,5 @@
           <box size="0.030 0.030 0.9144"/>
         </geometry>
-        <origin rpy="0 0 0" xyz="0 0 ${0.9144 / 2}"/>
+        <origin rpy="0 0 0" xyz="0 0.015 ${0.9144 / 2}"/>
       </visual>
       <collision>
@@ -46,5 +50,5 @@
           <box size="0.030 0.030 0.9144"/>
         </geometry>
-        <origin rpy="0 0 0" xyz="0 0 ${0.9144 / 2}"/>
+        <origin rpy="0 0 0" xyz="0 0.015 ${0.9144 / 2}"/>
       </collision>
     </link>
@@ -68,5 +72,5 @@
       <child link="camera_mount_2"/>
       <!-- edit origin of joints to change camera height -->
-      <origin xyz="0 0 0.8" rpy="${pi/2} 0 0"/>
+      <origin xyz="0.0 0.0 0.785" rpy="${pi/2} 0 0"/>
     </joint>
 <!-- 0.690875 -->
@@ -74,10 +78,10 @@
     <link name="camera_mount_3" />
     <xacro:sensor_d435 parent="camera_mount_3" use_nominal_extrinsics="$(arg use_nominal_extrinsics)" add_plug="$(arg add_plug)" use_mesh="$(arg use_mesh)">
-      <origin xyz="0 0 0" rpy="0 0 0"/>
+      <origin xyz="0.0245 0 -0.0125" rpy="0 0 0"/>
     </xacro:sensor_d435>
     <joint name="camera_mount_to_realsense_d435" type="fixed">
       <parent link="camera_mount_2"/>
       <child link="camera_mount_3"/>
-      <origin xyz="0.01 -0.025 0.3375" rpy="${pi/2} 0 ${3*pi/2}"/>
+      <origin xyz="0.0 0.0 0.3" rpy="${pi/2} 0 ${3*pi/2}"/>
     </joint>
     <material name="white">

File: workspace_test/urdf/synbio_env.urdf.xacro (robot description, xacro)
@@ -2,5 +2,19 @@
 <robot name="synbio_env" xmlns:xacro="http://ros.org/wiki/xacro">
   <xacro:include filename="$(find workspace_test)/urdf/env_macro.xacro"/>
-  <xacro:property name="table_height" value="0.845"/>
+  <xacro:include filename="$(find ur_description)/urdf/ur_macro.xacro"/>
+  <xacro:property name="table_height" value="0"/>
+  <!-- RIGHT -->
+  <xacro:property name="right_xyz" default="1.5748 0.508 ${table_height}"/>
+  <xacro:property name="right_rpy" default="0 0 ${pi}" />
+  <xacro:property name="right_tf_prefix" default="right_"/>
+  <!-- LEFT -->
+  <xacro:property name="left_xyz" default="0.9144 0.5588 ${table_height}" />
+  <xacro:property name="left_rpy" default="0 0 ${pi}" />
+  <xacro:property name="left_tf_prefix" default="left_"/>
+  <xacro:arg name="ur_type" default="ur3e"/>
+  <xacro:arg name="joint_limits_parameters_file" default="$(find ur_description)/config/$(arg ur_type)/joint_limits.yaml"/>
+  <xacro:arg name="kinematics_parameters_file" default="$(find ur_description)/config/$(arg ur_type)/default_kinematics.yaml"/>
+  <xacro:arg name="physical_parameters_file" default="$(find ur_description)/config/$(arg ur_type)/physical_parameters.yaml"/>
+  <xacro:arg name="visual_parameters_file" default="$(find ur_description)/config/$(arg ur_type)/visual_parameters.yaml"/>
   <link name="world"/>
   <!--This will create the scene where the robot is located in-->
@@ -10,3 +24,25 @@
       <origin xyz="0 0 ${table_height}" rpy="0 0 0" />
   </xacro:spawn_env>
+  <xacro:ur_robot
+    parent="world"
+    tf_prefix="${left_tf_prefix}"
+    name="left_$(arg ur_type)"
+    joint_limits_parameters_file="$(arg joint_limits_parameters_file)"
+    kinematics_parameters_file="$(arg kinematics_parameters_file)"
+    physical_parameters_file="$(arg physical_parameters_file)"
+    visual_parameters_file="$(arg visual_parameters_file)"
+    >
+    <origin xyz="${left_xyz}" rpy="${left_rpy}"/>
+  </xacro:ur_robot>
+  <xacro:ur_robot
+    parent="world"
+    tf_prefix="${right_tf_prefix}"
+    name="right_$(arg ur_type)"
+    joint_limits_parameters_file="$(arg joint_limits_parameters_file)"
+    kinematics_parameters_file="$(arg kinematics_parameters_file)"
+    physical_parameters_file="$(arg physical_parameters_file)"
+    visual_parameters_file="$(arg visual_parameters_file)"
+    >
+    <origin xyz="${right_xyz}" rpy="${right_rpy}"/>
+  </xacro:ur_robot>
 </robot>
