Commit message: Renamed moveit config setup

File: synbio_moveit_config/config/synbio_env.ros2_control.xacro (robot description, xacro)
@@ -1,92 +1,92 @@
 <?xml version="1.0"?>
 <robot xmlns:xacro="http://www.ros.org/wiki/xacro">
-    <xacro:macro name="my_robot_cell_ros2_control" params="name initial_positions_file">
+    <xacro:macro name="synbio_env_ros2_control" params="name initial_positions_file">
         <xacro:property name="initial_positions" value="${load_yaml(initial_positions_file)['initial_positions']}"/>
         <ros2_control name="${name}" type="system">
             <hardware>
                 <!-- By default, set up controllers for simulation. This won't work on real hardware -->
-                <plugin>mock_components/GenericSystem</plugin>
+                <plugin>ur_robot_driver/URPositionInterface</plugin>
             </hardware>
-            <joint name="ur3e1_shoulder_pan_joint">
+            <joint name="left_shoulder_pan_joint">
                 <command_interface name="position"/>
                 <state_interface name="position">
-                  <param name="initial_value">${initial_positions['ur3e1_shoulder_pan_joint']}</param>
+                  <param name="initial_value">${initial_positions['left_shoulder_pan_joint']}</param>
                 </state_interface>
                 <state_interface name="velocity"/>
             </joint>
-            <joint name="ur3e1_shoulder_lift_joint">
+            <joint name="left_shoulder_lift_joint">
                 <command_interface name="position"/>
                 <state_interface name="position">
-                  <param name="initial_value">${initial_positions['ur3e1_shoulder_lift_joint']}</param>
+                  <param name="initial_value">${initial_positions['left_shoulder_lift_joint']}</param>
                 </state_interface>
                 <state_interface name="velocity"/>
             </joint>
-            <joint name="ur3e1_elbow_joint">
+            <joint name="left_elbow_joint">
                 <command_interface name="position"/>
                 <state_interface name="position">
-                  <param name="initial_value">${initial_positions['ur3e1_elbow_joint']}</param>
+                  <param name="initial_value">${initial_positions['left_elbow_joint']}</param>
                 </state_interface>
                 <state_interface name="velocity"/>
             </joint>
-            <joint name="ur3e1_wrist_1_joint">
+            <joint name="left_wrist_1_joint">
                 <command_interface name="position"/>
                 <state_interface name="position">
-                  <param name="initial_value">${initial_positions['ur3e1_wrist_1_joint']}</param>
+                  <param name="initial_value">${initial_positions['left_wrist_1_joint']}</param>
                 </state_interface>
                 <state_interface name="velocity"/>
             </joint>
-            <joint name="ur3e1_wrist_2_joint">
+            <joint name="left_wrist_2_joint">
                 <command_interface name="position"/>
                 <state_interface name="position">
-                  <param name="initial_value">${initial_positions['ur3e1_wrist_2_joint']}</param>
+                  <param name="initial_value">${initial_positions['left_wrist_2_joint']}</param>
                 </state_interface>
                 <state_interface name="velocity"/>
             </joint>
-            <joint name="ur3e1_wrist_3_joint">
+            <joint name="left_wrist_3_joint">
                 <command_interface name="position"/>
                 <state_interface name="position">
-                  <param name="initial_value">${initial_positions['ur3e1_wrist_3_joint']}</param>
+                  <param name="initial_value">${initial_positions['left_wrist_3_joint']}</param>
                 </state_interface>
                 <state_interface name="velocity"/>
             </joint>
-            <joint name="ur3e2_shoulder_pan_joint">
+            <joint name="right_shoulder_pan_joint">
                 <command_interface name="position"/>
                 <state_interface name="position">
-                  <param name="initial_value">${initial_positions['ur3e2_shoulder_pan_joint']}</param>
+                  <param name="initial_value">${initial_positions['right_shoulder_pan_joint']}</param>
                 </state_interface>
                 <state_interface name="velocity"/>
             </joint>
-            <joint name="ur3e2_shoulder_lift_joint">
+            <joint name="right_shoulder_lift_joint">
                 <command_interface name="position"/>
                 <state_interface name="position">
-                  <param name="initial_value">${initial_positions['ur3e2_shoulder_lift_joint']}</param>
+                  <param name="initial_value">${initial_positions['right_shoulder_lift_joint']}</param>
                 </state_interface>
                 <state_interface name="velocity"/>
             </joint>
-            <joint name="ur3e2_elbow_joint">
+            <joint name="right_elbow_joint">
                 <command_interface name="position"/>
                 <state_interface name="position">
-                  <param name="initial_value">${initial_positions['ur3e2_elbow_joint']}</param>
+                  <param name="initial_value">${initial_positions['right_elbow_joint']}</param>
                 </state_interface>
                 <state_interface name="velocity"/>
             </joint>
-            <joint name="ur3e2_wrist_1_joint">
+            <joint name="right_wrist_1_joint">
                 <command_interface name="position"/>
                 <state_interface name="position">
-                  <param name="initial_value">${initial_positions['ur3e2_wrist_1_joint']}</param>
+                  <param name="initial_value">${initial_positions['right_wrist_1_joint']}</param>
                 </state_interface>
                 <state_interface name="velocity"/>
             </joint>
-            <joint name="ur3e2_wrist_2_joint">
+            <joint name="right_wrist_2_joint">
                 <command_interface name="position"/>
                 <state_interface name="position">
-                  <param name="initial_value">${initial_positions['ur3e2_wrist_2_joint']}</param>
+                  <param name="initial_value">${initial_positions['right_wrist_2_joint']}</param>
                 </state_interface>
                 <state_interface name="velocity"/>
             </joint>
-            <joint name="ur3e2_wrist_3_joint">
+            <joint name="right_wrist_3_joint">
                 <command_interface name="position"/>
                 <state_interface name="position">
-                  <param name="initial_value">${initial_positions['ur3e2_wrist_3_joint']}</param>
+                  <param name="initial_value">${initial_positions['right_wrist_3_joint']}</param>
                 </state_interface>
                 <state_interface name="velocity"/>

Commit message: Testing gripper addition and control

File: synbio_moveit_config/config/synbio_env.ros2_control.xacro (robot description, xacro)
@@ -6,5 +6,5 @@
             <hardware>
                 <!-- By default, set up controllers for simulation. This won't work on real hardware -->
-                <plugin>ur_robot_driver/URPositionInterface</plugin>
+                <plugin>mock_components/GenericSystem</plugin>
             </hardware>
             <joint name="left_shoulder_pan_joint">
@@ -92,4 +92,28 @@
                 <state_interface name="velocity"/>
             </joint>
+            <joint name="left_gripper_slider_1_joint">
+                <command_interface name="position"/>
+                <state_interface name="position">
+                  <param name="initial_value">${initial_positions['left_gripper_slider_1_joint']}</param>
+                </state_interface>
+            </joint>
+            <joint name="left_gripper_slider_2_joint">
+                <command_interface name="position"/>
+                <state_interface name="position">
+                  <param name="initial_value">${initial_positions['left_gripper_slider_2_joint']}</param>
+                </state_interface>
+            </joint>
+            <joint name="right_gripper_slider_1_joint">
+                <command_interface name="position"/>
+                <state_interface name="position">
+                  <param name="initial_value">${initial_positions['right_gripper_slider_1_joint']}</param>
+                </state_interface>
+            </joint>
+            <joint name="right_gripper_slider_2_joint">
+                <command_interface name="position"/>
+                <state_interface name="position">
+                  <param name="initial_value">${initial_positions['right_gripper_slider_2_joint']}</param>
+                </state_interface>
+            </joint>
         </ros2_control>
     </xacro:macro>

File: zimmer_description/urdf/ur3e.urdf.xacro (robot description, xacro)
@@ -2,5 +2,5 @@
 <robot name="ur3e_cell" xmlns:xacro="http://ros.org/wiki/xacro">
   <xacro:include filename="$(find zimmer_description)/urdf/zimmer_gripper_macro.xacro"/>
-  <xacro:include filename="$(find my_robot_cell_description)/urdf/my_robot_cell_macro.xacro"/>
+  <!-- <xacro:include filename="$(find my_robot_cell_description)/urdf/my_robot_cell_macro.xacro"/> -->
   <!-- end-effector prefix -->
   <xacro:arg name="prefix" default="zimmer_"/>
@@ -10,5 +10,5 @@
   <xacro:arg name="physical_parameters_file" default="$(find ur_description)/config/$(arg ur_type)/physical_parameters.yaml"/>
   <xacro:arg name="visual_parameters_file" default="$(find ur_description)/config/$(arg ur_type)/visual_parameters.yaml"/>
-  <link name="world"/>
+  <!-- <link name="world"/> -->
   <!--This will create the scene where the robot is located in-->
   <xacro:my_robot_cell
@@ -22,8 +22,9 @@
       <origin xyz="0 0 1" rpy="0 0 0" />
   </xacro:my_robot_cell>
+  <link name="world"/>
   <!-- end-effector -->
   <xacro:zimmer_gripper
       prefix="$(arg prefix)"
-      parent="$(arg ur_type)_tool0">
+      parent="world">
   </xacro:zimmer_gripper>
   <!-- Attach the gripper to the UR3e tool0 -->

File: zimmer_description/urdf/zimmer_gripper_macro.xacro (robot description, xacro)
@@ -2,4 +2,5 @@
 <robot name="zimmer_gripper" xmlns:xacro="http://www.ros.org/wiki/xacro">
   <xacro:include filename="$(find zimmer_description)/urdf/zimmer_description.xacro"/>
+  <!-- <xacro:arg name="parent" default="base_link"/> -->
   <xacro:macro name="zimmer_gripper" params="
     prefix
